File: hardware/hw_NANO33BLE/powercontrol.brd (EAGLE design)
At the start: 100 x 80 mm, 10 parts, among them Q1 IRF520, Q3 IRF520

Commit message: finished pcb
Parts:
- moved R2 15.2 mm to (47.0, 64.8)
- moved Q1 5.24 mm to (26.7, 47.0)
- moved Q3 5.24 mm to (26.7, 59.7)
- moved G1 3.59 mm to (29.2, 34.3), turned to 0 degrees
- moved S1 2.84 mm to (29.2, 24.1), turned to 90 degrees
Routing:
- net POWERGATE: track 0.00 -> 67.5 mm
- net 9V: track 0.00 -> 54.6 mm
- net D12: track 0.00 -> 41.9 mm
- net VIN: track 0.00 -> 24.0 mm
- net D11: track 0.00 -> 21.4 mm
- net GND2: track 0.00 -> 15.7 mm
- net DIODE_TO_RESISTOR: track 19.0 -> 3.81 mm
- net HAPTIC_GATE: track 8.67 -> 8.15 mm
Other:
- board size 100 x 80 mm -> 34 x 49.5 mm
- board text added: "Smart Gym Node"
